File: equatorial-mount.kicad_sch (KiCad schematic)
At the start: 1 part, among them U1 DRV8848

Commit message: working on schematic
Parts:
- added C1, C4: 10uF, Capacitor_SMD:C_1206_3216Metric, symbol Device:C_Small
- added C2, C5: 0.1uF, Capacitor_SMD:C_0603_1608Metric, symbol Device:C_Small
- added C3, C6: 2.2uF, Capacitor_SMD:C_0603_1608Metric, symbol Device:C_Small
- added J1, J2: 2MM_01x06_Socket, Connector_PinSocket_2.00mm:PinSocket_1x06_P2.00mm_Vertical, symbol Connector:Conn_01x06_Socket
- added J3: USB4110, Connector_USB:USB_C_Receptacle_GCT_USB4110, symbol Connector:USB_C_Receptacle_USB2.0_16P
- added R1, R2: 10K, Resistor_SMD:R_0603_1608Metric, symbol Device:R_US
- added R3, R4, R5, R6: 0.2, Resistor_SMD:R_1206_3216Metric, symbol Device:R_US
- added U2: ATmega32U4-A, Package_QFP:TQFP-44_10x10mm_P0.8mm, symbol MCU_Microchip_ATmega:ATmega32U4-A
- added U3: DRV8848, Package_SO:TSSOP-16-1EP_4.4x5mm_P0.65mm, symbol Driver_Motor:DRV8848
Connections:
- net +3.3V: now reaches U1.11 (VREF)
- net +3.3V: now also U1.14 (VINT), C3.1, C6.1, R1.1, R2.1, U3.11 (VREF), U3.14 (VINT)
- net +12V: now reaches U1.12 (VM)
- net +12V: now also C1.1, C2.1, C4.1, C5.1, U3.12 (VM)
- net GND: now reaches U1.13 (GND), U1.17 (GND)
- net GND: now also C1.2, C2.2, C3.2, C4.2, C5.2, C6.2, J3.A1 (GND), J3.A12 (GND), J3.B1 (GND), J3.B12 (GND), J3.S1 (SHIELD), R3.2, R4.2, R5.2, R6.2, U2.15 (GND), U2.23 (GND), U2.35 (GND), U2.43 (GND), U2.5 (UGND), U3.13 (GND), U3.17 (GND)
- net at U1.2 (AOUT1): now also J1.1 (Pin_1)
- net at U1.3 (AISEN): now also R3.1
- net at U1.4 (AOUT2): now also J1.3 (Pin_3)
- net at U1.5 (BOUT2): now also J1.6 (Pin_6)
- net at U1.6 (BISEN): now also R4.1
- net at U1.7 (BOUT1): now also J1.4 (Pin_4)
- net at U1.8 (~{FAULT}): now also R1.2
- new net: R2.2, U3.8 (~{FAULT})
- new net: R6.1, U3.3 (AISEN)
- new net: U2.14 (VCC), U2.34 (VCC)
- new net: U2.24 (AVCC), U2.44 (AVCC)
- new net: J2.1 (Pin_1), U3.2 (AOUT1)
- new net: J2.3 (Pin_3), U3.4 (AOUT2)
- new net: J2.4 (Pin_4), U3.7 (BOUT1)
- new net: J2.6 (Pin_6), U3.5 (BOUT2)
- new net: R5.1, U3.6 (BISEN)
- new net: J3.A4 (VBUS), J3.A9 (VBUS), J3.B4 (VBUS), J3.B9 (VBUS)
Other:
- moved on the sheet: U1

Commit message: sch
Parts:
- removed J3: USB4110, Connector_USB:USB_C_Receptacle_GCT_USB4110, symbol Connector:USB_C_Receptacle_USB2.0_16P
- removed U2: ATmega32U4-A, Package_QFP:TQFP-44_10x10mm_P0.8mm, symbol MCU_Microchip_ATmega:ATmega32U4-A
- added A1: RaspberryPi_Pico, Module:RaspberryPi_Pico_Common_Unspecified, symbol MCU_Module:RaspberryPi_Pico
- added J4, J5: SM04B-GHS-TB, Connector_JST:JST_GH_SM04B-GHS-TB_1x04-1MP_P1.25mm_Horizontal, symbol Connector:Conn_01x03_Pin
Connections:
- net +3.3V: now also A1.36 (3V3), J4.1 (Pin_1), J5.1 (Pin_1)
- net GND: now also A1.13 (GND), A1.18 (GND), A1.23 (GND), A1.28 (GND), A1.3 (GND), A1.38 (GND), A1.8 (GND), J4.3 (Pin_3), J5.3 (Pin_3)
- net at R2.2, U3.8 (~{FAULT}): now also A1.1 (GPIO0)
- net at U1.1 (~{SLEEP}): now also A1.22 (GPIO17)
- net at U1.10 (BIN2): now also A1.27 (GPIO21)
- net at U1.15 (AIN2): now also A1.25 (GPIO19)
- net at U1.16 (AIN1): now also A1.24 (GPIO18)
- net at R1.2, U1.8 (~{FAULT}): now also A1.21 (GPIO16)
- net at U1.9 (BIN1): now also A1.26 (GPIO20)
- net at U3.1 (~{SLEEP}): now also A1.2 (GPIO1)
- net at U3.10 (BIN2): now also A1.7 (GPIO5)
- net at U3.15 (AIN2): now also A1.5 (GPIO3)
- net at U3.16 (AIN1): now also A1.4 (GPIO2)
- net at U3.9 (BIN1): now also A1.6 (GPIO4)
- new net: A1.31 (GPIO26_ADC0), J5.2 (Pin_2)
- new net: A1.32 (GPIO27_ADC1), J4.2 (Pin_2)
Other:
- moved on the sheet: C1, C2, C3, C4, C5, C6, J1, J2, R1, R2, R3, R4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

Commit message: layout
Parts:
- removed C1: 10uF, Capacitor_SMD:C_1206_3216Metric, symbol Device:C_Small
- removed C2: 0.1uF, Capacitor_SMD:C_0603_1608Metric, symbol Device:C_Small
- removed C3: 2.2uF, Capacitor_SMD:C_0603_1608Metric, symbol Device:C_Small
- removed J1: 2MM_01x06_Socket, Connector_PinSocket_2.00mm:PinSocket_1x06_P2.00mm_Vertical, symbol Connector:Conn_01x06_Socket
- removed J4, J5: SM04B-GHS-TB, Connector_JST:JST_GH_SM04B-GHS-TB_1x04-1MP_P1.25mm_Horizontal, symbol Connector:Conn_01x03_Pin
- removed R1, R2: 10K, Resistor_SMD:R_0603_1608Metric, symbol Device:R_US
- removed R3, R4: 0.2, Resistor_SMD:R_1206_3216Metric, symbol Device:R_US
- removed U1: DRV8848, Package_SO:TSSOP-16-1EP_4.4x5mm_P0.65mm, symbol Driver_Motor:DRV8848
- added C1: 100uF, Capacitor_SMD:CP_Elec_10x7.7, symbol Device:C_Polarized_Small_US
- added C7: 2.2uF, Capacitor_SMD:C_0603_1608Metric, symbol Device:C_Small
- added C8: 0.1uF, Capacitor_SMD:C_0603_1608Metric, symbol Device:C_Small
- added C9: 10uF, Capacitor_SMD:C_1206_3216Metric, symbol Device:C_Small
- added H1, H2, H3, H4: M3, MountingHole:MountingHole_3.2mm_M3, symbol Mechanical:MountingHole
- added J3, J4: SM04B-GHS-TB, Connector_JST:JST_GH_SM04B-GHS-TB_1x04-1MP_P1.25mm_Horizontal, symbol Connector_Generic:Conn_01x04
- added J5: 2MM_01x06_Socket, Connector_PinSocket_2.00mm:PinSocket_1x06_P2.00mm_Vertical, symbol Connector:Conn_01x06_Socket
- added R7, R8: 0.2, Resistor_SMD:R_1206_3216Metric, symbol Device:R_US
- added TP1, TP2, TP3, TP4: TestPoint, jannett_footprints:TestPoint_Keystone_5016_Vias, symbol Connector:TestPoint
- added U4: DRV8848, Package_SO:TSSOP-16-1EP_4.4x5mm_P0.65mm, symbol Driver_Motor:DRV8848
Connections:
- net +12V: now also C1.1, C8.1, C9.1, TP1.1, U4.12 (VM)
- net +3.3V: now also C7.1, J3.1 (Pin_1), J4.1 (Pin_1), TP2.1, U4.11 (VREF), U4.14 (VINT)
- net GND: now also C1.2, C7.2, C8.2, C9.2, J3.4 (Pin_4), J4.4 (Pin_4), R7.2, R8.2, TP3.1, TP4.1, U4.13 (GND), U4.17 (GND)
- net at A1.10 (GPIO7): now also U4.1 (~{SLEEP})
- net at A1.11 (GPIO8): now also U4.16 (AIN1)
- net at A1.12 (GPIO9): now also U4.15 (AIN2)
- net at A1.14 (GPIO10): now also U4.9 (BIN1)
- net at A1.15 (GPIO11): now also U4.10 (BIN2)
- net at A1.31 (GPIO26_ADC0): now also J4.2 (Pin_2)
- net at A1.32 (GPIO27_ADC1): now also J3.2 (Pin_2)
- net at A1.9 (GPIO6): now also U4.8 (~{FAULT})
- net at J2.4 (Pin_4): now also U3.5 (BOUT2); no longer U3.7 (BOUT1)
- net at J2.6 (Pin_6): now also U3.7 (BOUT1); no longer U3.5 (BOUT2)
- new net: J5.1 (Pin_1), U4.2 (AOUT1)
- new net: R7.1, U4.3 (AISEN)
- new net: J5.3 (Pin_3), U4.4 (AOUT2)
- new net: J5.4 (Pin_4), U4.5 (BOUT2)
- new net: R8.1, U4.6 (BISEN)
- new net: J5.6 (Pin_6), U4.7 (BOUT1)
Other:
- moved on the sheet: A1, C4, C5, C6, J2, R5, R6, U3
