File: equatorial-mount.kicad_pcb (KiCad board)
At the start: 2 copper layers, 19 parts, among them J1 2MM_01x06_Socket, J2 2MM_01x06_Socket, J4 SM04B-GHS-TB, J5 SM04B-GHS-TB, U1 DRV8848, U3 DRV8848

Commit message: layout
Parts:
- removed C2: 0.1uF, Capacitor_SMD:C_0603_1608Metric
- removed C3: 2.2uF, Capacitor_SMD:C_0603_1608Metric
- removed J1: 2MM_01x06_Socket, Connector_PinSocket_2.00mm:PinSocket_1x06_P2.00mm_Vertical
- removed R1, R2: 10K, Resistor_SMD:R_0603_1608Metric
- removed R3, R4: 0.2, Resistor_SMD:R_1206_3216Metric
- removed U1: DRV8848, Package_SO:TSSOP-16-1EP_4.4x5mm_P0.65mm
- added C7: 2.2uF, Capacitor_SMD:C_0603_1608Metric, F.Cu at (122.4, 100.1)
- added C8: 0.1uF, Capacitor_SMD:C_0603_1608Metric, F.Cu at (122.2, 109.7)
- added C9: 10uF, Capacitor_SMD:C_1206_3216Metric, F.Cu at (122.2, 111.8)
- added H1: M3, MountingHole:MountingHole_3.2mm_M3, F.Cu at (110.2, 74.7)
- added H2: M3, MountingHole:MountingHole_3.2mm_M3, F.Cu at (156.5, 74.7)
- added H3: M3, MountingHole:MountingHole_3.2mm_M3, F.Cu at (110.2, 138.7)
- added H4: M3, MountingHole:MountingHole_3.2mm_M3, F.Cu at (156.5, 138.7)
- added J3: SM04B-GHS-TB, Connector_JST:JST_GH_SM04B-GHS-TB_1x04-1MP_P1.25mm_Horizontal, F.Cu at (156.2, 96.8)
- added R7: 0.2, Resistor_SMD:R_1206_3216Metric, F.Cu at (113.5, 103.6)
- added R8: 0.2, Resistor_SMD:R_1206_3216Metric, F.Cu at (113.5, 108.2)
- added TP1: TestPoint, jannett_footprints:TestPoint_Keystone_5016_Vias, F.Cu at (133.6, 136.9)
- added TP2: TestPoint, jannett_footprints:TestPoint_Keystone_5016_Vias, F.Cu at (156.0, 88.9)
- added TP3: TestPoint, jannett_footprints:TestPoint_Keystone_5016_Vias, F.Cu at (123.4, 136.9)
- added TP4: TestPoint, jannett_footprints:TestPoint_Keystone_5016_Vias, F.Cu at (156.0, 83.3)
- added U4: DRV8848, Package_SO:TSSOP-16-1EP_4.4x5mm_P0.65mm, F.Cu at (120.1, 104.9)
- C1: value 10uF -> 100uF; footprint Capacitor_SMD:C_1206_3216Metric -> Capacitor_SMD:CP_Elec_10x7.7
- J5: value SM04B-GHS-TB -> 2MM_01x06_Socket; footprint Connector_JST:JST_GH_SM04B-GHS-TB_1x04-1MP_P1.25mm_Horizontal -> Connector_PinSocket_2.00mm:PinSocket_1x06_P2.00mm_Vertical
- moved C1 82.8 mm to (117.3, 124.0), turned to 180 degrees
- moved J2 54.6 mm to (109.5, 81.9)
- moved R6 52.4 mm to (113.5, 84.1), turned to 180 degrees
- moved J5 52.4 mm to (109.2, 100.6)
- moved U3 52.2 mm to (120.1, 85.6)
- moved C4 51.4 mm to (122.2, 92.5), turned to 180 degrees
- moved R5 47.3 mm to (113.5, 89.2), turned to 180 degrees
- moved C5 45.8 mm to (122.2, 90.4), turned to 180 degrees
- moved J4 38.8 mm to (156.2, 107.2), turned to 90 degrees
- moved C6 37.1 mm to (122.4, 80.5), turned to 180 degrees
Connections:
- A1 pad 10: unconnected-(A1-GPIO7-Pad10) -> Net-(A1-GPIO7)
- A1 pad 11: unconnected-(A1-GPIO8-Pad11) -> Net-(A1-GPIO8)
- A1 pad 12: unconnected-(A1-GPIO9-Pad12) -> Net-(A1-GPIO9)
- A1 pad 14: unconnected-(A1-GPIO10-Pad14) -> Net-(A1-GPIO10)
- A1 pad 15: unconnected-(A1-GPIO11-Pad15) -> Net-(A1-GPIO11)
- A1 pad 21: Net-(A1-GPIO16) -> unconnected-(A1-GPIO16-Pad21)
- A1 pad 22: Net-(A1-GPIO17) -> unconnected-(A1-GPIO17-Pad22)
- A1 pad 24: Net-(A1-GPIO18) -> unconnected-(A1-GPIO18-Pad24)
- A1 pad 25: Net-(A1-GPIO19) -> unconnected-(A1-GPIO19-Pad25)
- A1 pad 26: Net-(A1-GPIO20) -> unconnected-(A1-GPIO20-Pad26)
- A1 pad 27: Net-(A1-GPIO21) -> unconnected-(A1-GPIO21-Pad27)
- A1 pad 9: unconnected-(A1-GPIO6-Pad9) -> Net-(A1-GPIO6)
- J4 pad 2: Net-(A1-GPIO27_ADC1) -> Net-(A1-GPIO26_ADC0)
- J4 pad 3: GND -> unconnected-(J4-Pin_3-Pad3)
- J4 pad 4: (no net) -> GND
- J5 pad 1: +3.3V -> Net-(J5-Pin_1)
- J5 pad 2: Net-(A1-GPIO26_ADC0) -> unconnected-(J5-Pin_2-Pad2)
- J5 pad 3: GND -> Net-(J5-Pin_3)
- J5 pad 4: (no net) -> Net-(J5-Pin_4)
- U3 pad 5: Net-(J2-Pin_6) -> Net-(J2-Pin_4)
- U3 pad 7: Net-(J2-Pin_4) -> Net-(J2-Pin_6)
Routing:
- net +3.3V: track 0.00 -> 33.7 mm
- net Net-(A1-GPIO26_ADC0): track 0.00 -> 16.0 mm
- net Net-(J2-Pin_6): track 0.00 -> 12.1 mm
- net Net-(J5-Pin_6): track 0.00 -> 11.2 mm
- net Net-(J2-Pin_1): track 0.00 -> 10.3 mm
- net Net-(J5-Pin_4): track 0.00 -> 10.3 mm
- net Net-(J5-Pin_3): track 0.00 -> 10.1 mm
- net Net-(J5-Pin_1): track 0.00 -> 9.92 mm
- net Net-(J2-Pin_4): track 0.00 -> 8.70 mm
- net Net-(A1-GPIO27_ADC1): track 0.00 -> 8.60 mm
- net Net-(J2-Pin_3): track 0.00 -> 8.14 mm
- net Net-(U3-BISEN): track 0.00 -> 5.16 mm
- net Net-(U4-BISEN): track 0.00 -> 4.51 mm
- net +12V: track 0.00 -> 3.24 mm
- net Net-(U4-AISEN): track 0.00 -> 3.02 mm
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- added copper zone on F.Cu, net +12V
- added copper zone on B.Cu, net GND
- added copper zone on F.Cu, net GND
Other:
- board outline added: 53.3 x 71.1 mm

Commit message: finished and gerbers
Parts:
- added G***: LOGO, jannett_footprints:saturn, B.Cu at (143.5, 130.3)
Routing:
- net +3.3V: track 33.7 -> 99.1 mm, vias 0 -> 2
- net Net-(A1-GPIO0): track 0.00 -> 50.7 mm
- net Net-(A1-GPIO6): track 0.00 -> 24.4 mm, vias 0 -> 1
- net Net-(A1-GPIO1): track 0.00 -> 16.4 mm
- net Net-(A1-GPIO7): track 0.00 -> 14.9 mm, vias 0 -> 1
- net Net-(A1-GPIO5): track 0.00 -> 10.4 mm, vias 0 -> 1
- net Net-(A1-GPIO11): track 0.00 -> 9.81 mm, vias 0 -> 1
- net Net-(A1-GPIO4): track 0.00 -> 8.38 mm, vias 0 -> 1
- net Net-(A1-GPIO8): track 0.00 -> 8.38 mm, vias 0 -> 1
- net Net-(A1-GPIO9): track 0.00 -> 7.89 mm, vias 0 -> 1
- net Net-(A1-GPIO10): track 0.00 -> 7.60 mm, vias 0 -> 1
- net GND: track 0.00 -> 7.40 mm, vias 0 -> 73
- net Net-(A1-GPIO2): track 0.00 -> 7.16 mm
- net Net-(A1-GPIO3): track 0.00 -> 6.38 mm
Other:
- board text added: "12V"
- board text added: "3.3V"
- board text added: "Azimuth"
- board text added: "Elevation"
- board text added: "Equatorial Mount Controller V01"
- board text added: "GND"
- board text added: "Jannett W"
- board text added: "{dblquote}Do not look at stars as bright spots only. Try to take in the vastness of the universe.{dblquote} - Maria Mitchell, Astronomer"
